Commit message: Add torque plot for dynamics squatting in the PyBullet Giving some initial CoM offset to avoid falling of the robot Fixing the Torso joint to avoid rotation

File: models/a1_alpha_biped_corrected_mass/urdf/A1_alpha_biped_concept_urdf.urdf (robot description, URDF)
Before this commit: robot A1_alpha_biped_concept_urdf, 17 links, 16 joints
Joints:
- joint Torso_Yaw_DOF: limit lower=-3.1416 upper=3.1416 effort=90 velocity=16.441 -> lower=-0.1 upper=0.1 effort=0.0 velocity=16.441

Commit message: Smoothening squatting (touch down and squat) and fully lock Torso-yaw link

File: models/a1_alpha_biped_corrected_mass/urdf/A1_alpha_biped_concept_urdf.urdf (robot description, URDF)
Before this commit: robot A1_alpha_biped_concept_urdf, 17 links, 16 joints
Joints:
- joint Torso_Yaw_DOF: limit lower=-0.1 upper=0.1 effort=0.0 velocity=16.441 -> lower=0.0 upper=0.0 effort=0.0 velocity=16.441
